File: WaterLevel - Display/WaterLevel.sch (KiCad schematic (older format))
At the start: 58 parts, among them P1 PWR_SW, P2 PROBE, P3 AC 12V, P4 PUMP, P5 ALARM, Q1 2N2222, Q2 2N2222, U1 LM324N, U2 LM7812CT, U3 LM324N, U4 LM324N

Commit message: Display
Parts:
- removed C1: CP, Capacitors_ThroughHole:C_Radial_D5_L11_P2.5, symbol CP
- removed C2: CP, Capacitors_ThroughHole:C_Axial_D13_L31_P38, symbol CP
- removed D1, D8: 1N4007, Diodes_ThroughHole:Diode_DO-41_SOD81_Vertical_KathodeUp, symbol D
- removed D2: PUMP_LED, LEDs:LED-5MM, symbol LED
- removed D3, D4, D5, D6: D, Diodes_ThroughHole:Diode_DO-41_SOD81_Vertical_KathodeUp, symbol D
- removed D7: PWR_LED, LEDs:LED-5MM, symbol LED
- removed D9: ALRM_LED, LEDs:LED-5MM, symbol LED
- removed F1: FUSE, Fuse_Holders_and_Fuses:Fuseholder5x20_horiz_open_Schurter_0031_8201, symbol FUSE
- removed P1: PWR_SW, Sockets_MOLEX_KK-System:Socket_MOLEX-KK-RM3-96mm_Lock_2pin_straight, symbol CONN_01X02
- removed P2: PROBE, Sockets_MOLEX_KK-System:Socket_MOLEX-KK-RM3-96mm_Lock_3pin_straight, symbol CONN_01X03
- removed P3: AC 12V, Sockets_MOLEX_KK-System:Socket_MOLEX-KK-RM3-96mm_Lock_2pin_straight, symbol CONN_01X02
- removed P4: PUMP, Sockets_MOLEX_KK-System:Socket_MOLEX-KK-RM3-96mm_Lock_2pin_straight, symbol CONN_01X02
- removed P5: ALARM, Sockets_MOLEX_KK-System:Socket_MOLEX-KK-RM3-96mm_Lock_3pin_straight, symbol CONN_01X03
- removed Q1, Q2: 2N2222, TO_SOT_Packages_THT:TO-18_3Pin, symbol Q_NPN_EBC
- removed R1, R2, R3, R4, R5: R, Resistors_ThroughHole:Resistor_Horizontal_RM7mm, symbol R
- removed RL1, RL2: 12V/2A, Relays_ThroughHole:Relay_SPDT_Schrack-RT1_RM5mm, symbol RM50-xx11
- removed RV1, RV2: POT, Potentiometers:Potentiometer_Trimmer-Piher_PT15-V15_horizontal, symbol POT
- removed RV3: ALRM_LVL, Potentiometers:Potentiometer_Trimmer-Piher_PT15-V15_horizontal, symbol POT
- removed U1: LM324N, Housings_DIP:DIP-14_W7.62mm_LongPads, symbol LM324N
- removed U2: LM7812CT, Power_Integrations:TO-220, symbol LM7812CT
- added P1: DISPLAY, Sockets_MOLEX_KK-System:Socket_MOLEX-KK-RM2-54mm_Lock_3pin_straight, symbol CONN_01X03
- renumbered D10 to D1, D11 to D2, D12 to D3, D13 to D4, D14 to D5, D15 to D6, D16 to D7, D17 to D8, R6 to R1, R15 to R10, R16 to R11, R17 to R12, R18 to R13, R19 to R14, R20 to R15, R7 to R2, R8 to R3, R9 to R4, R10 to R5, R11 to R6, R12 to R7, R13 to R8, R14 to R9, RV4 to RV1, RV5 to RV2, U3 to U1, U4 to U2
Connections:
- net +12V: now also P1.1 (P1)
- net GNDPWR: now also P1.3 (P3)
- net VProbe: no longer names the net of U1.13 (-), U1.2 (-), U1.6 (-), U1.9 (-), U2.13 (-), U2.2 (-), U2.6 (-), U2.9 (-)
- net VProbe: now also P1.2 (P2)
- no-connect marks 13 -> 12
Other:
- note removed: "Alimentation montage"
- note removed: "Connecteur Sonde"
- note removed: "Etage de commande de pompe"
- note removed: "Etage de notification alarme"
- moved on the sheet: D1, D2, D3, D4, D5, D6, D7, D8, R1, R10, R11, R12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

Commit message: Updates
Parts:
- removed P1: DISPLAY, Sockets_MOLEX_KK-System:Socket_MOLEX-KK-RM2-54mm_Lock_3pin_straight, symbol CONN_01X03
- added P1: GND, Wire_Pads:SolderWirePad_single_1mmDrill, symbol CONN_01X01
- added P2: VIN, Wire_Pads:SolderWirePad_single_1mmDrill, symbol CONN_01X01
- added P3: +12V, Wire_Pads:SolderWirePad_single_1mmDrill, symbol CONN_01X01
Connections:
- net +12V: now also P3.1 (P1)
- net GNDPWR: now also P1.1 (P1)
- net at U1.13 (-), U1.2 (-), U1.6 (-)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: now also P2.1 (P1)
Changed lines of the file:
@@
 Wire Wire Line
 	4250 3150 4250 3400
-$Comp
-L CONN_01X03 P1
-U 1 1 57741236
-P 2800 3350
-F 0 "P1" H 2800 3550 50  0000 C CNN
-F 1 "DISPLAY" V 2900 3350 50  0000 C CNN
-F 2 "Sockets_MOLEX_KK-System:Socket_MOLEX-KK-RM2-54mm_Lock_3pin_straight" H 2800 3350 50  0001 C CNN
-F 3 "" H 2800 3350 50  0000 C CNN
-	1    2800 3350
-	-1   0    0    1
-$EndComp
 Wire Wire Line
-	3000 3250 3000 2100
+	3000 2100 3000 3250
 Connection ~ 3500 2100
 Wire Wire Line
-	3300 2500 3300 3350
+	3300 2500 3300 3450
 Wire Wire Line
-	3300 3350 3000 3350
-Wire Wire Line
-	3000 3450 3450 3450
-Wire Wire Line
-	3450 3450 3450 4600
+	3450 3650 3450 4600
 Connection ~ 3950 4600
 $Comp
@@
 	3300 4050 3450 4050
 Connection ~ 3450 4050
+$Comp
+L CONN_01X01 P1
+U 1 1 578174C6
+P 2800 3250
+F 0 "P1" H 2800 3350 50  0000 C CNN
+F 1 "GND" V 2900 3250 50  0000 C CNN
+F 2 "Wire_Pads:SolderWirePad_single_1mmDrill" H 2800 3250 50  0001 C CNN
+F 3 "" H 2800 3250 50  0000 C CNN
+	1    2800 3250
+	-1   0    0    1
+$EndComp
+$Comp
+L CONN_01X01 P2
+U 1 1 57817552
+P 2800 3450
+F 0 "P2" H 2800 3550 50  0000 C CNN
+F 1 "VIN" V 2900 3450 50  0000 C CNN
+F 2 "Wire_Pads:SolderWirePad_single_1mmDrill" H 2800 3450 50  0001 C CNN
+F 3 "" H 2800 3450 50  0000 C CNN
+	1    2800 3450
+	-1   0    0    1
+$EndComp
+$Comp
+L CONN_01X01 P3
+U 1 1 578175D8
+P 2800 3650
+F 0 "P3" H 2800 3750 50  0000 C CNN
+F 1 "+12V" V 2900 3650 50  0000 C CNN
+F 2 "Wire_Pads:SolderWirePad_single_1mmDrill" H 2800 3650 50  0001 C CNN
+F 3 "" H 2800 3650 50  0000 C CNN
+	1    2800 3650
+	-1   0    0    1
+$EndComp
+Wire Wire Line
+	3000 3650 3450 3650
+Wire Wire Line
+	3300 3450 3000 3450
 $EndSCHEMATC

Commit message: Final version of display
Parts:
- removed RV1: LVL, Potentiometers:Potentiometer_Trimmer-Piher_PT15-V15_horizontal, symbol POT
- removed RV2: LVH, Potentiometers:Potentiometer_Trimmer-Piher_PT15-V15_horizontal, symbol POT
- added R16: RLVL, Resistors_ThroughHole:Resistor_Horizontal_RM7mm, symbol R
- added R17: RLVH, Resistors_ThroughHole:Resistor_Horizontal_RM7mm, symbol R
Connections:
- net +12V: now also R17.1
- net GNDPWR: now also R16.2
- net at R9.1: now also U1.14; no longer U1.7
- net at R11.1: now also U1.7; no longer U1.14
- net at R13.1: now also U2.14; no longer U2.7
- net at R15.1: now also U2.7; no longer U2.14
- net at P2.1 (P1), U1.2 (-), U1.9 (-)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: now also U1.13 (-), U1.6 (-), U2.13 (-), U2.6 (-); no longer U1.13 (-), U1.6 (-), U2.13 (-), U2.6 (-)
- net at R1.2, U1.3 (+): now also R16.1
- net at R1.1, R2.2: now also U1.12 (+); no longer U1.5 (+)
- net at R3.1, R4.2: now also U1.5 (+); no longer U1.12 (+)
- net at R5.1, R6.2: now also U2.12 (+); no longer U2.5 (+)
- net at R7.1: now also U2.5 (+), R17.2; no longer U2.12 (+)
Changed lines of the file:
@@
 encoding utf-8
 Sheet 1 1
-Title ""
-Date ""
-Rev ""
-Comp ""
+Title "Sonde niveau d'eau - Ecran"
+Date "2016-07-16"
+Rev "1.0"
+Comp "Chatons Corp"
 Comment1 ""
 Comment2 ""
@@
 $Comp
 L LM324N U1
-U 2 1 57714913
+U 4 1 57714913
 P 4500 3000
 F 0 "U1" H 4550 3200 50  0000 C CNN
@@
 F 2 "Housings_DIP:DIP-14_W7.62mm_LongPads" H 4450 3100 50  0001 C CNN
 F 3 "" H 4550 3200 50  0000 C CNN
-	2    4500 3000
+	4    4500 3000
 	0    1    1    0
 $EndComp
@@
 $Comp
 L LM324N U1
-U 4 1 577161FF
+U 2 1 577161FF
 P 5600 3000
 F 0 "U1" H 5650 3200 50  0000 C CNN
@@
 F 2 "Housings_DIP:DIP-14_W7.62mm_LongPads" H 5550 3100 50  0001 C CNN
 F 3 "" H 5650 3200 50  0000 C CNN
-	4    5600 3000
+	2    5600 3000
 	0    1    1    0
 $EndComp
@@
 $Comp
 L LM324N U2
-U 2 1 577164A5
+U 4 1 577164A5
 P 6700 3000
 F 0 "U2" H 6750 3200 50  0000 C CNN
@@
 F 2 "Housings_DIP:DIP-14_W7.62mm_LongPads" H 6650 3100 50  0001 C CNN
 F 3 "" H 6750 3200 50  0000 C CNN
-	2    6700 3000
+	4    6700 3000
 	0    1    1    0
 $EndComp
@@
 $Comp
 L LM324N U2
-U 4 1 5771659C
+U 2 1 5771659C
 P 7800 3000
 F 0 "U2" H 7850 3200 50  0000 C CNN
@@
 F 2 "Housings_DIP:DIP-14_W7.62mm_LongPads" H 7750 3100 50  0001 C CNN
 F 3 "" H 7850 3200 50  0000 C CNN
-	4    7800 3000
+	2    7800 3000
 	0    1    1    0
 $EndComp
@@
 	7700 2500 7700 2700
 Connection ~ 7150 2500
-$Comp
-L POT RV1
-U 1 1 5771843C
-P 3750 2100
-F 0 "RV1" H 3750 2020 50  0000 C CNN
-F 1 "LVL" H 3750 2100 50  0000 C CNN
-F 2 "Potentiometers:Potentiometer_Trimmer-Piher_PT15-V15_horizontal" H 3750 2100 50  0001 C CNN
-F 3 "" H 3750 2100 50  0000 C CNN
-	1    3750 2100
-	-1   0    0    1
-$EndComp
 Wire Wire Line
 	3500 2150 3500 2100
 Wire Wire Line
 	3000 2100 3600 2100
-Wire Wire Line
-	3750 2250 3900 2250
-Wire Wire Line
-	3900 2250 3900 2100
 Wire Wire Line
 	3900 2100 4250 2100
@@
 Wire Wire Line
 	7900 2100 7900 2700
-$Comp
-L POT RV2
-U 1 1 577196E3
-P 8150 2100
-F 0 "RV2" H 8150 2020 50  0000 C CNN
-F 1 "LVH" H 8150 2100 50  0000 C CNN
-F 2 "Potentiometers:Potentiometer_Trimmer-Piher_PT15-V15_horizontal" H 8150 2100 50  0001 C CNN
-F 3 "" H 8150 2100 50  0000 C CNN
-	1    8150 2100
-	-1   0    0    1
-$EndComp
-Wire Wire Line
-	8400 4600 8400 1950
-Wire Wire Line
-	8150 2250 8300 2250
-Wire Wire Line
-	8300 2250 8300 2100
+Wire Wire Line
+	8400 1950 8400 4600
 Wire Wire Line
 	8300 2100 8400 2100
@@
 Wire Wire Line
 	3300 3450 3000 3450
+$Comp
+L R R16
+U 1 1 578A0DD6
+P 3750 2100
+F 0 "R16" V 3830 2100 50  0000 C CNN
+F 1 "RLVL" V 3750 2100 50  0000 C CNN
+F 2 "Resistors_ThroughHole:Resistor_Horizontal_RM7mm" V 3680 2100 50  0001 C CNN
+F 3 "" H 3750 2100 50  0000 C CNN
+	1    3750 2100
+	0    1    1    0
+$EndComp
+$Comp
+L R R17
+U 1 1 578A10D0
+P 8150 2100
+F 0 "R17" V 8230 2100 50  0000 C CNN
+F 1 "RLVH" V 8150 2100 50  0000 C CNN
+F 2 "Resistors_ThroughHole:Resistor_Horizontal_RM7mm" V 8080 2100 50  0001 C CNN
+F 3 "" H 8150 2100 50  0000 C CNN
+	1    8150 2100
+	0    1    1    0
+$EndComp
 $EndSCHEMATC
