File: WaterLevel - Display/WaterLevel.kicad_pcb (KiCad board)
At the start: 2 copper layers, 30 parts, among them P1 GND, P2 VIN, P3 +12V, U1 LM324N, U2 LM324N

Commit message: Final version of display
Parts:
- removed RV1: LVL, Potentiometers:Potentiometer_Trimmer-Piher_PT15-V15_horizontal
- removed RV2: LVH, Potentiometers:Potentiometer_Trimmer-Piher_PT15-V15_horizontal
- added R16: RLVL, Resistors_ThroughHole:Resistor_Horizontal_RM7mm, F.Cu at (50.9, 81.7)
- added R17: RLVH, Resistors_ThroughHole:Resistor_Horizontal_RM7mm, F.Cu at (31.9, 22.1)
- added na: na, Wire_Pads:Big_Square_Pad_3mm_1mmDrill, F.Cu at (36.6, 54.1)
- added via11: via, Wire_Pads:Big_Square_Pad_3mm_1mmDrill, F.Cu at (36.6, 66.7)
- added via12: via, Wire_Pads:Big_Square_Pad_3mm_1mmDrill, F.Cu at (43.6, 66.4)
- added via13: via, Wire_Pads:Big_Square_Pad_3mm_1mmDrill, F.Cu at (48.4, 66.4)
- added via21: via, Wire_Pads:Big_Square_Pad_3mm_1mmDrill, F.Cu at (43.4, 51.4)
- added via22: via, Wire_Pads:Big_Square_Pad_3mm_1mmDrill, F.Cu at (48.2, 51.4)
- added via25: via, Wire_Pads:Big_Square_Pad_3mm_1mmDrill, F.Cu at (40.1, 89.9)
- added via35: via, Wire_Pads:Big_Square_Pad_3mm_1mmDrill, F.Cu at (48.4, 90.2)
- moved D8 189.9 mm to (22.6, 22.1), turned to 0 degrees
- moved D7 179.0 mm to (22.6, 31.6), turned to 0 degrees
- moved R15 174.7 mm to (29.1, 26.9), turned to 180 degrees
- moved D6 168.2 mm to (22.6, 41.1), turned to 0 degrees
- moved R7 167.2 mm to (35.1, 25.4), turned to 270 degrees
- moved R14 164.0 mm to (29.1, 36.4), turned to 180 degrees
- moved D5 157.5 mm to (22.6, 50.6), turned to 0 degrees
- moved R6 157.0 mm to (32.1, 32.9), turned to 270 degrees
- moved R13 153.4 mm to (29.1, 45.9), turned to 180 degrees
- moved D4 146.9 mm to (22.6, 60.1), turned to 0 degrees
- moved R5 146.5 mm to (32.1, 43.4), turned to 270 degrees
- moved R12 142.9 mm to (29.1, 55.4), turned to 180 degrees
- moved D3 136.3 mm to (22.6, 69.7), turned to 0 degrees
- moved R11 132.5 mm to (29.1, 64.9), turned to 180 degrees
- moved R4 129.9 mm to (33.4, 56.4), turned to 270 degrees
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Connections:
- R7 pad 1: Net-(R7-Pad1) -> Net-(R17-Pad2)
- U1 pad 12: Net-(R3-Pad1) -> Net-(R1-Pad1)
- U1 pad 14: Net-(R11-Pad1) -> Net-(R9-Pad1)
- U1 pad 5: Net-(R1-Pad1) -> Net-(R3-Pad1)
- U1 pad 7: Net-(R9-Pad1) -> Net-(R11-Pad1)
- U2 pad 12: Net-(R7-Pad1) -> Net-(R5-Pad1)
- U2 pad 14: Net-(R15-Pad1) -> Net-(R13-Pad1)
- U2 pad 5: Net-(R5-Pad1) -> Net-(R17-Pad2)
- U2 pad 7: Net-(R13-Pad1) -> Net-(R15-Pad1)
Routing:
- net Net-(P2-Pad1): track 0.00 -> 97.4 mm, vias 0 -> 2
- net +12V: track 44.4 -> 115.9 mm
- net GNDPWR: track 0.00 -> 69.3 mm
- net Net-(R1-Pad2): track 58.0 -> 29.3 mm, vias 0 -> 2
- net Net-(R7-Pad1): track 28.0 -> 0.00 mm
- net Net-(R17-Pad2): track 0.00 -> 27.8 mm
- net Net-(R15-Pad1): track 42.0 -> 17.7 mm
- net Net-(R1-Pad1): track 24.1 -> 10.2 mm, vias 2 -> 0
- net Net-(R13-Pad1): track 20.8 -> 9.23 mm
- net Net-(R4-Pad1): track 24.9 -> 36.4 mm, vias 0 -> 2
- net Net-(R8-Pad1): track 37.3 -> 26.1 mm, vias 2 -> 0
- net Net-(R2-Pad1): track 20.4 -> 9.70 mm
- net Net-(R11-Pad1): track 35.6 -> 26.3 mm
- net Net-(R5-Pad1): track 18.5 -> 9.28 mm
- net Net-(R9-Pad1): track 20.5 -> 11.5 mm
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Other:
- board outline added: 36 x 80.8 mm

Commit message: Updates
Parts:
- added REF**: SolderWirePad_single_2mmDrill, Wire_Pads:SolderWirePad_single_2mmDrill, F.Cu at (50.8, 22.0)
- added REF**: SolderWirePad_single_2mmDrill, Wire_Pads:SolderWirePad_single_2mmDrill, F.Cu at (50.8, 95.0)
- added REF**: SolderWirePad_single_2mmDrill, Wire_Pads:SolderWirePad_single_2mmDrill, F.Cu at (44.6, 59.6)
- moved P3 0.60 mm to (36.6, 93.4)
- moved P2 0.50 mm to (41.4, 93.4)
- moved P1 0.40 mm to (47.2, 93.4)
Routing:
- added copper zone on B.Cu, net GNDPWR
Other:
- board text added: "AG 2016"
Changed lines of the file:
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@@
     (links 54)
     (no_connects 0)
-    (area 91.124999 46.688 127.97512 128.475001)
+    (area 18.524999 17.065 68.301453 107.300001)
     (thickness 1.6)
-    (drawings 4)
+    (drawings 7)
     (tracks 167)
     (zones 0)
-    (modules 38)
+    (modules 41)
     (nets 28)
   )
@@
     (0 F.Cu signal)
     (31 B.Cu signal)
-    (32 B.Adhes user)
-    (33 F.Adhes user)
-    (34 B.Paste user)
-    (35 F.Paste user)
-    (36 B.SilkS user)
     (37 F.SilkS user)
-    (38 B.Mask user)
-    (39 F.Mask user)
-    (40 Dwgs.User user)
-    (41 Cmts.User user)
-    (42 Eco1.User user)
-    (43 Eco2.User user)
     (44 Edge.Cuts user)
     (45 Margin user)
-    (46 B.CrtYd user)
-    (47 F.CrtYd user)
-    (48 B.Fab user)
-    (49 F.Fab user)
   )
   (setup
@@
     (trace_clearance 0.2)
     (zone_clearance 0.508)
-    (zone_45_only no)
+    (zone_45_only yes)
     (trace_min 0.2)
     (segment_width 0.2)
@@
     (mod_text_size 1 1)
     (mod_text_width 0.15)
-    (pad_size 2 2)
-    (pad_drill 0.5)
+    (pad_size 4.50088 4.50088)
+    (pad_drill 1.99898)
     (pad_to_mask_clearance 0.2)
     (aux_axis_origin 0 0)
@@
   )
   (module Wire_Pads:SolderWirePad_single_1mmDrill (layer F.Cu)
-    (at 46.8 93.4 90)
+    (at 47.2 93.4 90)
     (fp_text reference P1 (at -4.5 0 180) (layer F.SilkS)
       (effects (font (size 1 1) (thickness 0.15)))
@@
   )
   (module Wire_Pads:SolderWirePad_single_1mmDrill (layer F.Cu)
-    (at 41.9 93.4)
+    (at 41.4 93.4)
     (fp_text reference P2 (at 0 4.5) (layer F.SilkS)
       (effects (font (size 1 1) (thickness 0.15)))
@@
   )
   (module Wire_Pads:SolderWirePad_single_1mmDrill (layer F.Cu)
-    (at 37.2 93.4)
+    (at 36.6 93.4)
     (fp_text reference P3 (at 0 4.5) (layer F.SilkS)
       (effects (font (size 1 1) (thickness 0.15)))
@@
     (descr "Resistor, Axial,  RM 7.62mm, 1/3W,")
     (tags "Resistor Axial RM 7.62mm 1/3W R3")
-    (fp_text reference R16 (at 4.05892 -3.50012 270) (layer F.SilkS)
+    (fp_text reference R16 (at 3.75 -0.1 270) (layer F.SilkS)
       (effects (font (size 1 1) (thickness 0.15)))
     )
@@
     )
     (pad 1 thru_hole circle (at 0 0) (size 2 2) (drill 0.5) (layers *.Cu *.Mask F.SilkS))
+  )
+  (module Wire_Pads:SolderWirePad_single_2mmDrill (layer F.Cu)
+    (at 50.8 22)
+    (fp_text reference REF** (at 0 -3.81) (layer F.SilkS) hide
+      (effects (font (size 1 1) (thickness 0.15)))
+    )
+    (fp_text value SolderWirePad_single_2mmDrill (at -0.635 3.81) (layer F.Fab) hide
+      (effects (font (size 1 1) (thickness 0.15)))
+    )
+    (pad 1 thru_hole circle (at 0 0) (size 4.50088 4.50088) (drill 1.99898) (layers *.Cu *.Mask F.SilkS))
+  )
+  (module Wire_Pads:SolderWirePad_single_2mmDrill (layer F.Cu)
+    (at 50.8 95)
+    (fp_text reference REF** (at 0 -3.81) (layer F.SilkS) hide
+      (effects (font (size 1 1) (thickness 0.15)))
+    )
+    (fp_text value SolderWirePad_single_2mmDrill (at -0.635 3.81) (layer F.Fab) hide
+      (effects (font (size 1 1) (thickness 0.15)))
+    )
+    (pad 1 thru_hole circle (at 0 0) (size 4.50088 4.50088) (drill 1.99898) (layers *.Cu *.Mask F.SilkS))
+  )
+  (module Wire_Pads:SolderWirePad_single_2mmDrill (layer F.Cu)
+    (at 44.6 59.6)
+    (fp_text reference REF** (at 0 -3.81) (layer F.SilkS) hide
+      (effects (font (size 1 1) (thickness 0.15)))
+    )
+    (fp_text value SolderWirePad_single_2mmDrill (at -0.635 3.81) (layer F.Fab) hide
+      (effects (font (size 1 1) (thickness 0.15)))
+    )
+    (pad 1 thru_hole circle (at 0 0) (size 4.50088 4.50088) (drill 1.99898) (layers *.Cu))
+  )
+  (gr_text "AG 2016" (at 41.2 25.4) (layer B.Cu)
+    (effects (font (size 1.5 1.2) (thickness 0.3)) (justify mirror))
+  )
+  (dimension 80.800248 (width 0.3) (layer F.SilkS)
+    (gr_text "80.800 mm" (at 61.651453 58.414731 89.85817905) (layer F.SilkS)
+      (effects (font (size 1.5 1.5) (thickness 0.3)))
+    )
+    (feature1 (pts (xy 55.8 18) (xy 63.101449 18.018073)))
+    (feature2 (pts (xy 55.6 98.8) (xy 62.901449 98.818073)))
+    (crossbar (pts (xy 60.201457 98.81139) (xy 60.401457 18.01139)))
+    (arrow1a (pts (xy 60.401457 18.01139) (xy 60.985088 19.139342)))
+    (arrow1b (pts (xy 60.401457 18.01139) (xy 59.81225 19.136439)))
+    (arrow2a (pts (xy 60.201457 98.81139) (xy 60.790664 97.686341)))
+    (arrow2b (pts (xy 60.201457 98.81139) (xy 59.617826 97.683438)))
+  )
+  (dimension 36 (width 0.3) (layer F.SilkS)
+    (gr_text "36.000 mm" (at 36.6 105.95) (layer F.SilkS)
+      (effects (font (size 1.5 1.5) (thickness 0.3)))
+    )
+    (feature1 (pts (xy 54.6 100.2) (xy 54.6 107.3)))
+    (feature2 (pts (xy 18.6 100.2) (xy 18.6 107.3)))
+    (crossbar (pts (xy 18.6 104.6) (xy 54.6 104.6)))
+    (arrow1a (pts (xy 54.6 104.6) (xy 53.473496 105.186421)))
+    (arrow1b (pts (xy 54.6 104.6) (xy 53.473496 104.013579)))
+    (arrow2a (pts (xy 18.6 104.6) (xy 19.726504 105.186421)))
+    (arrow2b (pts (xy 18.6 104.6) (xy 19.726504 104.013579)))
   )
   (gr_line (start 18.6 18) (end 18.6 98.8) (angle 90) (layer Edge.Cuts) (width 0.15))
@@
   (segment (start 39.52 22.15) (end 38.4 22.15) (width 1) (layer B.Cu) (net 27))
   (segment (start 38.4 22.15) (end 35.15 25.4) (width 1) (layer B.Cu) (net 27))
+  (zone (net 2) (net_name GNDPWR) (layer B.Cu) (hatch edge 0.508)
+    (connect_pads yes (clearance 0.508))
+    (min_thickness 0.508)
+    (fill yes (arc_segments 16) (thermal_gap 0.508) (thermal_bridge_width 0.508))
+    (polygon
+      (pts
+        (xy 54.6 98.8) (xy 18.6 98.8) (xy 18.6 18) (xy 54.6 18) (xy 54.6 98.8)
+      )
+    )
+  )
 )
