File: WaterLevel - Main/WaterLevel.kicad_pcb (KiCad board)
At the start: 2 copper layers, 58 parts, among them P1 PWR_SW, P2 PROBE, P3 AC 12V, P4 PUMP, P5 ALARM, Q1 2N2222, Q2 2N2222, U1 LM324N, U2 LM7812CT, U3 LM324N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

Commit message: Base PCB
Parts:
- removed D10: LN1, LEDs:LED-5MM
- removed D11: LN2, LEDs:LED-5MM
- removed D12: LN3, LEDs:LED-5MM
- removed D13: LN4, LEDs:LED-5MM
- removed D14: LN5, LEDs:LED-5MM
- removed D15: LN6, LEDs:LED-5MM
- removed D16: LN7, LEDs:LED-5MM
- removed D17: LN8, LEDs:LED-5MM
- removed R10, R11, R12, R13, R14, R15, R16, R17, R18, R19, R20, R6, R7, R8, R9: R, Resistors_ThroughHole:Resistor_Horizontal_RM7mm
- removed RV4: LVL, Potentiometers:Potentiometer_Trimmer-Piher_PT15-V15_horizontal
- removed RV5: LVH, Potentiometers:Potentiometer_Trimmer-Piher_PT15-V15_horizontal
- removed U3, U4: LM324N, Housings_DIP:DIP-14_W7.62mm_LongPads
- added P6: ALARM, Sockets_MOLEX_KK-System:Socket_MOLEX-KK-RM3-96mm_Lock_3pin_straight, F.Cu at (247.4, 103.1)
- C1: value CP -> 10uF
- C2: value CP -> 2200uF
- D1, D4, D8: footprint Diodes_ThroughHole:Diode_DO-41_SOD81_Vertical_KathodeUp -> Diodes_ThroughHole:Diode_DO-41_SOD81_Horizontal_RM10
- D2: value PUMP_LED -> 1N4007; footprint LEDs:LED-5MM -> Diodes_ThroughHole:Diode_DO-41_SOD81_Horizontal_RM10
- D3, D6: value D -> 1N4007; footprint Diodes_ThroughHole:Diode_DO-41_SOD81_Vertical_KathodeUp -> Diodes_ThroughHole:Diode_DO-41_SOD81_Horizontal_RM10
- D5: value D -> PWR; footprint Diodes_ThroughHole:Diode_DO-41_SOD81_Vertical_KathodeUp -> LEDs:LED-5MM
- D7: value PWR_LED -> PUMP
- D9: value ALRM_LED -> ALRM
- F1: value FUSE -> 1A 12V
- P1: value PWR_SW -> PWRSW
- P3: value AC 12V -> DISPLAY; footprint Sockets_MOLEX_KK-System:Socket_MOLEX-KK-RM3-96mm_Lock_2pin_straight -> Sockets_MOLEX_KK-System:Socket_MOLEX-KK-RM3-96mm_Lock_3pin_straight
- P4: value PUMP -> 12VAC
- P5: value ALARM -> PUMP; footprint Sockets_MOLEX_KK-System:Socket_MOLEX-KK-RM3-96mm_Lock_3pin_straight -> Sockets_MOLEX_KK-System:Socket_MOLEX-KK-RM3-96mm_Lock_2pin_straight
- R1, R2, R4: value R -> 2.2k
- R3, R5: value R -> 10k
- RV1: value POT -> LVL2
- RV2: value POT -> LVL1
- RV3: value ALRM_LVL -> ALRM
- U1: value LM324N -> LM7812CT; footprint Housings_DIP:DIP-14_W7.62mm_LongPads -> Power_Integrations:TO-220
- U2: value LM7812CT -> LM324N; footprint Power_Integrations:TO-220 -> Housings_DIP:DIP-14_W7.62mm_LongPads
- moved F1 225.2 mm to (250.2, 143.3), turned to 180 degrees
- moved D3 165.0 mm to (223.5, 135.1)
- moved D4 159.5 mm to (213.4, 143.0), turned to 0 degrees
- moved P3 159.4 mm to (184.2, 143.5), turned to 0 degrees
- moved D5 150.3 mm to (197.9, 131.3), turned to 180 degrees
- moved D6 150.1 mm to (203.2, 77.5), turned to 270 degrees
- moved P1 143.2 mm to (205.7, 123.2), turned to 90 degrees
- moved C2 136.5 mm to (213.1, 118.6), turned to 0 degrees
- moved C1 108.5 mm to (200.2, 135.9), turned to 0 degrees
- moved D7 104.2 mm to (209.6, 92.7), turned to 180 degrees
- moved R2 87.7 mm to (199.4, 85.1)
- moved P2 82.5 mm to (170.7, 143.5), turned to 0 degrees
- moved U2 74.9 mm to (176.5, 94.5), turned to 270 degrees
- moved U1 71.5 mm to (202.7, 143.0), turned to 180 degrees
- moved R1 65.4 mm to (195.1, 146.6), turned to 90 degrees
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Connections:
- D1 pad 1: +12V -> Net-(D1-Pad1)
- D2 pad 1: Net-(D1-Pad2) -> Net-(D2-Pad1)
- D2 pad 2: Net-(D2-Pad2) -> Net-(D1-Pad1)
- D3 pad 1: Net-(D3-Pad1) -> Net-(D1-Pad2)
- D3 pad 2: Net-(D3-Pad2) -> GNDPWR
- D4 pad 1: Net-(D3-Pad1) -> GNDPWR
- D4 pad 2: Net-(D4-Pad2) -> Net-(D2-Pad1)
- D5 pad 2: Net-(D3-Pad2) -> Net-(D5-Pad2)
- D6 pad 1: GNDPWR -> +12V
- D6 pad 2: Net-(D4-Pad2) -> Net-(D6-Pad2)
- D7 pad 1: GNDPWR -> Net-(D6-Pad2)
- F1 pad 2: Net-(D4-Pad2) -> Net-(D2-Pad1)
- P1 pad 1: Net-(D3-Pad1) -> Net-(D1-Pad1)
- P3 pad 1: Net-(D3-Pad2) -> +12V
- P3 pad 2: Net-(F1-Pad1) -> VProbe
- P4 pad 1: Net-(P4-Pad1) -> Net-(D1-Pad2)
- P4 pad 2: GNDPWR -> Net-(F1-Pad1)
- P5 pad 2: Net-(P5-Pad2) -> GNDPWR
- Q1 pad 3: Net-(D1-Pad2) -> Net-(D6-Pad2)
- R1 pad 2: Net-(D2-Pad2) -> Net-(D5-Pad2)
- RL1 pad 11: Net-(P4-Pad1) -> Net-(P5-Pad1)
- RL1 pad A2: Net-(D1-Pad2) -> Net-(D6-Pad2)
- RL2 pad 11: Net-(P5-Pad3) -> Net-(P6-Pad3)
- RL2 pad 12: Net-(P5-Pad1) -> Net-(P6-Pad1)
- RL2 pad 14: Net-(P5-Pad2) -> Net-(P6-Pad2)
- U1 pad 1: Net-(R3-Pad1) -> +12VA
- U1 pad 2: Net-(RV1-Pad2) -> GNDPWR
- U1 pad 3: Net-(RV2-Pad2) -> +12V
- U2 pad 1: +12VA -> Net-(R3-Pad1)
- U2 pad 2: GNDPWR -> Net-(RV1-Pad2)
- U2 pad 3: +12V -> Net-(RV2-Pad2)

Commit message: PCB implem
Parts:
- moved P2 1.78 mm to (168.9, 143.5)
Routing:
- net GNDPWR: track 0.00 -> 215.0 mm
- net +12V: track 0.00 -> 129.3 mm
- net VProbe: track 0.00 -> 65.7 mm
- net +12VA: track 0.00 -> 62.9 mm
- net Net-(P5-Pad1): track 0.00 -> 35.1 mm
- net Net-(P6-Pad1): track 0.00 -> 34.4 mm
- net Net-(D1-Pad1): track 0.00 -> 30.8 mm
- net Net-(P6-Pad3): track 0.00 -> 29.9 mm
- net Net-(D1-Pad2): track 0.00 -> 28.3 mm
- net Net-(D8-Pad2): track 0.00 -> 24.1 mm
- net Net-(P6-Pad2): track 0.00 -> 22.8 mm
- net Net-(F1-Pad1): track 0.00 -> 18.6 mm
- net Net-(D6-Pad2): track 0.00 -> 12.5 mm
- net Net-(R5-Pad1): track 0.00 -> 12.5 mm
- net Net-(R3-Pad1): track 0.00 -> 11.4 mm
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Other:
- net class Default: trace_width 0.25 -> 1
- net class Power: trace_width 1 -> 1.5

Commit message: Updates
Parts:
- removed F1: 1A 12V, Fuse_Holders_and_Fuses:Fuseholder5x20_horiz_open_Schurter_0031_8201
- added P10: PM-, Wire_Pads:Big_Square_Pad_3mm_1mmDrill, F.Cu at (250.8, 86.8)
- added P11: ALNC, Wire_Pads:Big_Square_Pad_3mm_1mmDrill, F.Cu at (225.2, 86.8)
- added P12: ALNO, Wire_Pads:Big_Square_Pad_3mm_1mmDrill, F.Cu at (233.2, 86.8)
- added P13: ALC, Wire_Pads:Big_Square_Pad_3mm_1mmDrill, F.Cu at (229.2, 86.8)
- added P7: 12Vac, Wire_Pads:Big_Square_Pad_3mm_1mmDrill, F.Cu at (246.2, 129.8)
- added P8: 12Vac, Wire_Pads:Big_Square_Pad_3mm_1mmDrill, F.Cu at (246.2, 125.5)
- added P9: PM+, Wire_Pads:Big_Square_Pad_3mm_1mmDrill, F.Cu at (243.8, 86.8)
- P1: value PWRSW -> PR+; footprint Sockets_MOLEX_KK-System:Socket_MOLEX-KK-RM3-96mm_Lock_2pin_straight -> Wire_Pads:Big_Square_Pad_3mm_1mmDrill
- P2: value PROBE -> PRv; footprint Sockets_MOLEX_KK-System:Socket_MOLEX-KK-RM3-96mm_Lock_3pin_straight -> Wire_Pads:Big_Square_Pad_3mm_1mmDrill
- P3: value DISPLAY -> PR-; footprint Sockets_MOLEX_KK-System:Socket_MOLEX-KK-RM3-96mm_Lock_3pin_straight -> Wire_Pads:Big_Square_Pad_3mm_1mmDrill
- P4: value 12VAC -> DS+; footprint Sockets_MOLEX_KK-System:Socket_MOLEX-KK-RM3-96mm_Lock_2pin_straight -> Wire_Pads:Big_Square_Pad_3mm_1mmDrill
- P5: value PUMP -> DSv; footprint Sockets_MOLEX_KK-System:Socket_MOLEX-KK-RM3-96mm_Lock_2pin_straight -> Wire_Pads:Big_Square_Pad_3mm_1mmDrill
- P6: value ALARM -> DS-; footprint Sockets_MOLEX_KK-System:Socket_MOLEX-KK-RM3-96mm_Lock_3pin_straight -> Wire_Pads:Big_Square_Pad_3mm_1mmDrill
- moved P5 87.0 mm to (173.0, 128.0), turned to 0 degrees
- moved P6 83.4 mm to (167.8, 128.0), turned to 0 degrees
- moved P4 69.0 mm to (178.2, 128.0), turned to 0 degrees
- moved C2 53.3 mm to (171.8, 85.0), turned to 270 degrees
- moved RV1 51.1 mm to (199.8, 134.8), turned to 0 degrees
- moved RV3 39.1 mm to (184.2, 87.5), turned to 270 degrees
- moved RV2 32.4 mm to (194.0, 118.8), turned to 180 degrees
- moved R1 31.8 mm to (216.8, 123.2), turned to 0 degrees
- moved D5 30.4 mm to (227.5, 124.8), turned to 90 degrees
- moved P1 29.5 mm to (178.2, 134.0), turned to 0 degrees
- moved R3 28.6 mm to (204.8, 115.2)
- moved U2 22.6 mm to (197.2, 103.5)
- moved D1 21.1 mm to (232.4, 121.6)
- moved D2 21.1 mm to (242.3, 129.7)
- moved D4 21.1 mm to (232.1, 133.3)
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Connections:
- D1 pad 1: Net-(D1-Pad1) -> +12VA
- D2 pad 2: Net-(D1-Pad1) -> +12VA
- P1 pad 1: Net-(D1-Pad1) -> +12V
- P2 pad 1: +12V -> VProbe
- P3 pad 1: +12V -> GNDPWR
- P4 pad 1: Net-(D1-Pad2) -> +12V
- P5 pad 1: Net-(P5-Pad1) -> VProbe
- P6 pad 1: Net-(P6-Pad1) -> GNDPWR
- RL1 pad 11: Net-(P5-Pad1) -> Net-(P9-Pad1)
- RL2 pad 11: Net-(P6-Pad3) -> Net-(P13-Pad1)
- RL2 pad 12: Net-(P6-Pad1) -> Net-(P11-Pad1)
- RL2 pad 14: Net-(P6-Pad2) -> Net-(P12-Pad1)
- U2 pad 1: Net-(R3-Pad1) -> Net-(R5-Pad1)
- U2 pad 12: VProbe -> Net-(RV2-Pad2)
- U2 pad 13: Net-(RV3-Pad2) -> Net-(RV1-Pad2)
- U2 pad 14: Net-(R5-Pad1) -> Net-(R3-Pad1)
- U2 pad 2: Net-(RV1-Pad2) -> Net-(RV3-Pad2)
- U2 pad 3: Net-(RV2-Pad2) -> VProbe
Routing:
- net GNDPWR: track 215.0 -> 348.0 mm, vias 0 -> 4
- net +12VA: track 62.9 -> 154.0 mm
- net VProbe: track 65.7 -> 124.2 mm
- net +12V: track 129.3 -> 186.7 mm
- net Net-(RV3-Pad2): track 0.00 -> 54.0 mm
- net Net-(P12-Pad1): track 0.00 -> 39.5 mm
- net Net-(P13-Pad1): track 0.00 -> 38.9 mm
- net Net-(P11-Pad1): track 0.00 -> 38.1 mm
- net Net-(RV2-Pad2): track 0.00 -> 36.0 mm
- net Net-(P5-Pad1): track 35.1 -> 0.00 mm
- net Net-(P6-Pad1): track 34.4 -> 0.00 mm
- net Net-(R3-Pad1): track 11.4 -> 45.8 mm
- net Net-(D1-Pad1): track 30.8 -> 0.00 mm
- net Net-(P6-Pad3): track 29.9 -> 0.00 mm
- net Net-(P6-Pad2): track 22.8 -> 0.00 mm
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
Commit message: Updates
Parts:
- added R6: 10k, Resistors_ThroughHole:Resistor_Horizontal_RM7mm, F.Cu at (192.6, 115.0)
- added REF**: SolderWirePad_single_0-8mmDrill, Wire_Pads:SolderWirePad_single_0-8mmDrill, F.Cu at (221.8, 132.0)
- added REF**: SolderWirePad_single_0-8mmDrill, Wire_Pads:SolderWirePad_single_0-8mmDrill, F.Cu at (214.4, 132.0)
- added REF**: SolderWirePad_single_0-8mmDrill, Wire_Pads:SolderWirePad_single_0-8mmDrill, F.Cu at (208.6, 89.6)
- added REF**: SolderWirePad_single_2mmDrill, Wire_Pads:SolderWirePad_single_2mmDrill, F.Cu at (251.2, 85.4)
- added REF**: SolderWirePad_single_0-8mmDrill, Wire_Pads:SolderWirePad_single_0-8mmDrill, F.Cu at (201.6, 89.6)
- added REF**11: SolderWirePad_single_2mmDrill, Wire_Pads:SolderWirePad_single_2mmDrill, F.Cu at (165.8, 85.4)
- added REF**15: SolderWirePad_single_2mmDrill, Wire_Pads:SolderWirePad_single_2mmDrill, F.Cu at (251.2, 138.6)
- added REF**21: SolderWirePad_single_2mmDrill, Wire_Pads:SolderWirePad_single_2mmDrill, F.Cu at (165.8, 138.6)
- C2: footprint Capacitors_ThroughHole:C_Axial_D13_L31_P38 -> Capacitors_ThroughHole:C_Radial_D14_L25_P5
- RL1, RL2: footprint Relays_ThroughHole:Relay_SPDT_Schrack-RT1_RM5mm -> relays:Relay_1RT_Hongfa_HF33F
- RV1, RV2, RV3: footprint Potentiometers:Potentiometer_Trimmer-Piher_PT15-V15_horizontal -> Potentiometers:Potentiometer_Trimmer-Piher_PT10-V10_horizontal
- moved P12 32.7 mm to (249.8, 115.0)
- moved P13 31.0 mm to (249.8, 110.0)
- moved P11 30.6 mm to (249.8, 105.0)
- moved C2 29.9 mm to (169.2, 114.8), turned to 0 degrees
- moved P10 11.9 mm to (249.8, 98.6)
- moved P9 9.14 mm to (249.8, 93.6)
- moved P7 3.58 mm to (249.8, 130.2)
- moved P8 3.56 mm to (249.8, 125.2)
- moved RV2 3.26 mm to (193.8, 122.0)
- moved RV3 3.15 mm to (186.6, 89.6)
- moved RV1 2.76 mm to (200.8, 132.2)
Connections:
- RV2 pad 2: Net-(RV2-Pad2) -> Net-(R6-Pad1)
- RV2 pad 3: Net-(R3-Pad1) -> Net-(R6-Pad1)
- U2 pad 12: Net-(RV2-Pad2) -> Net-(R6-Pad1)
Routing:
- net Net-(RV2-Pad2): track 36.0 -> 0.00 mm
- net Net-(R3-Pad1): track 45.8 -> 10.9 mm
- net GNDPWR: track 348.0 -> 315.0 mm
- net Net-(P12-Pad1): track 39.5 -> 10.2 mm
- net Net-(R6-Pad1): track 0.00 -> 24.3 mm
- net Net-(P11-Pad1): track 38.1 -> 14.0 mm
- net Net-(P9-Pad1): track 12.9 -> 32.9 mm
- net Net-(P13-Pad1): track 38.9 -> 19.5 mm
- net Net-(RV3-Pad2): track 54.0 -> 43.2 mm
- net VProbe: track 124.2 -> 116.5 mm
- net Net-(RL1-Pad12): track 7.62 -> 0.00 mm
- net Net-(D2-Pad1): track 7.92 -> 11.5 mm
- net Net-(D1-Pad2): track 7.44 -> 11.0 mm
- net +12V: track 186.7 -> 183.2 mm
- net +12VA: track 154.0 -> 156.0 mm
- added copper zone on B.Cu, net GNDPWR
Other:
- board outline added: 91 x 58.8 mm
