File: WaterLevel - Main/WaterLevel.sch (KiCad schematic (older format))
At the start: 58 parts, among them P1 PWR_SW, P2 PROBE, P3 AC 12V, P4 PUMP, P5 ALARM, Q1 2N2222, Q2 2N2222, U1 LM324N, U2 LM7812CT, U3 LM324N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

Commit message: Base PCB
Parts:
- removed D10: LN1, LEDs:LED-5MM, symbol LED
- removed D11: LN2, LEDs:LED-5MM, symbol LED
- removed D12: LN3, LEDs:LED-5MM, symbol LED
- removed D13: LN4, LEDs:LED-5MM, symbol LED
- removed D14: LN5, LEDs:LED-5MM, symbol LED
- removed D15: LN6, LEDs:LED-5MM, symbol LED
- removed D16: LN7, LEDs:LED-5MM, symbol LED
- removed D17: LN8, LEDs:LED-5MM, symbol LED
- removed R10, R11, R12, R13, R14, R15, R16, R17, R18, R19, R20, R6, R7, R8, R9: R, Resistors_ThroughHole:Resistor_Horizontal_RM7mm, symbol R
- removed RV4: LVL, Potentiometers:Potentiometer_Trimmer-Piher_PT15-V15_horizontal, symbol POT
- removed RV5: LVH, Potentiometers:Potentiometer_Trimmer-Piher_PT15-V15_horizontal, symbol POT
- removed U3, U4: LM324N, Housings_DIP:DIP-14_W7.62mm_LongPads, symbol LM324N
- added P3: DISPLAY, Sockets_MOLEX_KK-System:Socket_MOLEX-KK-RM3-96mm_Lock_3pin_straight, symbol CONN_01X03
- C1: value CP -> 10uF
- C2: value CP -> 2200uF
- D1: renamed from D3; value D -> 1N4007; footprint Diodes_ThroughHole:Diode_DO-41_SOD81_Vertical_KathodeUp -> Diodes_ThroughHole:Diode_DO-41_SOD81_Horizontal_RM10
- D2: renamed from D4; value D -> 1N4007; footprint Diodes_ThroughHole:Diode_DO-41_SOD81_Vertical_KathodeUp -> Diodes_ThroughHole:Diode_DO-41_SOD81_Horizontal_RM10
- D3: renamed from D5; value D -> 1N4007; footprint Diodes_ThroughHole:Diode_DO-41_SOD81_Vertical_KathodeUp -> Diodes_ThroughHole:Diode_DO-41_SOD81_Horizontal_RM10
- D4: renamed from D6; footprint Diodes_ThroughHole:Diode_DO-41_SOD81_Vertical_KathodeUp -> Diodes_ThroughHole:Diode_DO-41_SOD81_Horizontal_RM10
- D5: renamed from D7; value PWR_LED -> PWR
- D6: renamed from D1; footprint Diodes_ThroughHole:Diode_DO-41_SOD81_Vertical_KathodeUp -> Diodes_ThroughHole:Diode_DO-41_SOD81_Horizontal_RM10
- D7: renamed from D2; value PUMP_LED -> PUMP
- D8: footprint Diodes_ThroughHole:Diode_DO-41_SOD81_Vertical_KathodeUp -> Diodes_ThroughHole:Diode_DO-41_SOD81_Horizontal_RM10
- D9: value ALRM_LED -> ALRM
- F1: value FUSE -> 1A 12V
- P1: value PWR_SW -> PWRSW
- P4: renamed from P3; value AC 12V -> 12VAC
- R1: renamed from R2; value R -> 2.2k
- R2: renamed from R1; value R -> 2.2k
- R3, R5: value R -> 10k
- R4: value R -> 2.2k
- RV1: value POT -> LVL2
- RV2: value POT -> LVL1
- RV3: value ALRM_LVL -> ALRM
- renumbered P4 to P5, P5 to P6, U2 to U1, U1 to U2
Connections:
- net +12V: now also P3.1 (P1)
- net GNDPWR: now also D3.2 (A), P3.3 (P3); no longer D3.1 (K)
- net VProbe: now also U2.12 (+), P3.2 (P2); no longer U2.5 (+)
- net at D1.2 (A), P4.1 (P1): now also D3.1 (K); no longer D3.2 (A)
- net at D1.1 (K), P1.1 (P1): now also D2.2 (A); no longer D2.1 (K)
- net at D4.2 (A), F1.2: now also D2.1 (K); no longer D2.2 (A)
- net at RV3.2: now also U2.13 (-); no longer U2.6 (-)
- net at R5.1: now also U2.14; no longer U2.7
- no-connect marks 13 -> 1
Other:
- note added: "Connecteur Visu"
- note removed: "Etage visualisation"
- moved on the sheet: D6, D7, D8, D9, P5, P6, Q1, Q2, R2, R3, R4, R5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

Commit message: Updates
Parts:
- removed F1: 1A 12V, Fuse_Holders_and_Fuses:Fuseholder5x20_horiz_open_Schurter_0031_8201, symbol FUSE
- removed P1: PWRSW, Sockets_MOLEX_KK-System:Socket_MOLEX-KK-RM3-96mm_Lock_2pin_straight, symbol CONN_01X02
- removed P2: PROBE, Sockets_MOLEX_KK-System:Socket_MOLEX-KK-RM3-96mm_Lock_3pin_straight, symbol CONN_01X03
- removed P3: DISPLAY, Sockets_MOLEX_KK-System:Socket_MOLEX-KK-RM3-96mm_Lock_3pin_straight, symbol CONN_01X03
- removed P4: 12VAC, Sockets_MOLEX_KK-System:Socket_MOLEX-KK-RM3-96mm_Lock_2pin_straight, symbol CONN_01X02
- removed P5: PUMP, Sockets_MOLEX_KK-System:Socket_MOLEX-KK-RM3-96mm_Lock_2pin_straight, symbol CONN_01X02
- removed P6: ALARM, Sockets_MOLEX_KK-System:Socket_MOLEX-KK-RM3-96mm_Lock_3pin_straight, symbol CONN_01X03
- added P1: PR+, Wire_Pads:Big_Square_Pad_3mm_1mmDrill, symbol CONN_01X01
- added P10: PM-, Wire_Pads:Big_Square_Pad_3mm_1mmDrill, symbol CONN_01X01
- added P11: ALNC, Wire_Pads:Big_Square_Pad_3mm_1mmDrill, symbol CONN_01X01
- added P12: ALNO, Wire_Pads:Big_Square_Pad_3mm_1mmDrill, symbol CONN_01X01
- added P13: ALC, Wire_Pads:Big_Square_Pad_3mm_1mmDrill, symbol CONN_01X01
- added P2: PRv, Wire_Pads:Big_Square_Pad_3mm_1mmDrill, symbol CONN_01X01
- added P3: PR-, Wire_Pads:Big_Square_Pad_3mm_1mmDrill, symbol CONN_01X01
- added P4: DS+, Wire_Pads:Big_Square_Pad_3mm_1mmDrill, symbol CONN_01X01
- added P5: DSv, Wire_Pads:Big_Square_Pad_3mm_1mmDrill, symbol CONN_01X01
- added P6: DS-, Wire_Pads:Big_Square_Pad_3mm_1mmDrill, symbol CONN_01X01
- added P7, P8: 12Vac, Wire_Pads:Big_Square_Pad_3mm_1mmDrill, symbol CONN_01X01
- added P9: PM+, Wire_Pads:Big_Square_Pad_3mm_1mmDrill, symbol CONN_01X01
Connections:
- net +12V: now also P1.1 (P1), P4.1 (P1)
- net +12VA: now also D1.1 (K), D2.2 (A)
- net GNDPWR: now also P10.1 (P1), P3.1 (P1), P6.1 (P1)
- net VProbe: now also U2.3 (+), P2.1 (P1), P5.1 (P1); no longer U2.12 (+)
- net at D1.2 (A), D3.1 (K): now also P8.1 (P1)
- net at D2.1 (K), D4.2 (A): now also P7.1 (P1)
- net at R3.1, RV2.3: now also U2.14; no longer U2.1
- net at RV1.2: now also U2.13 (-); no longer U2.2 (-)
- net at RV2.2: now also U2.12 (+); no longer U2.3 (+)
- net at RL1.11: now also P9.1 (P1)
- net at RV3.2: now also U2.2 (-); no longer U2.13 (-)
- net at R5.1: now also U2.1; no longer U2.14
- net at RL2.11: now also P13.1 (P1)
- net at RL2.12: now also P11.1 (P1)
- net at RL2.14: now also P12.1 (P1)

Commit message: Updates
Parts:
- added R6: 10k, Resistors_ThroughHole:Resistor_Horizontal_RM7mm, symbol R
- C2: footprint Capacitors_ThroughHole:C_Axial_D13_L31_P38 -> Capacitors_ThroughHole:C_Radial_D14_L25_P5
- RL1, RL2: footprint Relays_ThroughHole:Relay_SPDT_Schrack-RT1_RM5mm -> relays:Relay_1RT_Hongfa_HF33F
- RV1, RV2, RV3: footprint Potentiometers:Potentiometer_Trimmer-Piher_PT15-V15_horizontal -> Potentiometers:Potentiometer_Trimmer-Piher_PT10-V10_horizontal
Connections:
- net at RV2.2, U2.12 (+): now also RV2.3, R6.1
- net at R3.1, U2.14: now also R6.2; no longer RV2.3
Other:
- moved on the sheet: RV2
Changed lines of the file:
@@
 F 0 "RL1" H 5500 4550 50  0000 L CNN
 F 1 "12V/2A" H 5500 4450 50  0000 L CNN
-F 2 "Relays_ThroughHole:Relay_SPDT_Schrack-RT1_RM5mm" H 5050 4400 50  0001 C CNN
+F 2 "relays:Relay_1RT_Hongfa_HF33F" H 5050 4400 50  0001 C CNN
 F 3 "" H 5050 4400 50  0000 C CNN
 	1    5050 4400
@@
 F 0 "C2" H 2875 1950 50  0000 L CNN
 F 1 "2200uF" H 2875 1750 50  0000 L CNN
-F 2 "Capacitors_ThroughHole:C_Axial_D13_L31_P38" H 2888 1700 50  0001 C CNN
+F 2 "Capacitors_ThroughHole:C_Radial_D14_L25_P5" H 2888 1700 50  0001 C CNN
 F 3 "" H 2850 1850 50  0000 C CNN
 	1    2850 1850
@@
 F 0 "RV1" H 2750 4470 50  0000 C CNN
 F 1 "LVL2" H 2750 4550 50  0000 C CNN
-F 2 "Potentiometers:Potentiometer_Trimmer-Piher_PT15-V15_horizontal" H 2750 4550 50  0001 C CNN
+F 2 "Potentiometers:Potentiometer_Trimmer-Piher_PT10-V10_horizontal" H 2750 4550 50  0001 C CNN
 F 3 "" H 2750 4550 50  0000 C CNN
 	1    2750 4550
@@
 L POT RV2
 U 1 1 57712C85
-P 3050 5250
-F 0 "RV2" H 3050 5170 50  0000 C CNN
-F 1 "LVL1" H 3050 5250 50  0000 C CNN
-F 2 "Potentiometers:Potentiometer_Trimmer-Piher_PT15-V15_horizontal" H 3050 5250 50  0001 C CNN
-F 3 "" H 3050 5250 50  0000 C CNN
-	1    3050 5250
-	1    0    0    -1
-$EndComp
-Wire Wire Line
-	3050 5100 3050 4350
+P 2850 5250
+F 0 "RV2" H 2850 5170 50  0000 C CNN
+F 1 "LVL1" H 2850 5250 50  0000 C CNN
+F 2 "Potentiometers:Potentiometer_Trimmer-Piher_PT10-V10_horizontal" H 2850 5250 50  0001 C CNN
+F 3 "" H 2850 5250 50  0000 C CNN
+	1    2850 5250
+	1    0    0    -1
+$EndComp
 Wire Wire Line
 	3050 4350 3200 4350
@@
 VProbe
 Wire Wire Line
-	2550 5250 2900 5250
+	2550 5250 2700 5250
 Wire Wire Line
 	4250 4000 4250 4050
@@
 Connection ~ 4850 4800
 Connection ~ 4500 4800
-Wire Wire Line
-	3950 5250 3200 5250
 Wire Wire Line
 	4850 5500 4850 5250
@@
 F 0 "RL2" H 5550 6500 50  0000 L CNN
 F 1 "12V/2A" H 5550 6400 50  0000 L CNN
-F 2 "Relays_ThroughHole:Relay_SPDT_Schrack-RT1_RM5mm" H 5100 6350 50  0001 C CNN
+F 2 "relays:Relay_1RT_Hongfa_HF33F" H 5100 6350 50  0001 C CNN
 F 3 "" H 5100 6350 50  0000 C CNN
 	1    5100 6350
@@
 F 0 "RV3" H 2900 6770 50  0000 C CNN
 F 1 "ALRM" H 2900 6700 50  0000 C CNN
-F 2 "Potentiometers:Potentiometer_Trimmer-Piher_PT15-V15_horizontal" H 2900 6850 50  0001 C CNN
+F 2 "Potentiometers:Potentiometer_Trimmer-Piher_PT10-V10_horizontal" H 2900 6850 50  0001 C CNN
 F 3 "" H 2900 6850 50  0000 C CNN
 	1    2900 6850
@@
 	1    0    0    -1
 $EndComp
+$Comp
+L R R6
+U 1 1 578D43E7
+P 3650 5250
+F 0 "R6" V 3730 5250 50  0000 C CNN
+F 1 "10k" V 3650 5250 50  0000 C CNN
+F 2 "Resistors_ThroughHole:Resistor_Horizontal_RM7mm" V 3580 5250 50  0001 C CNN
+F 3 "" H 3650 5250 50  0000 C CNN
+	1    3650 5250
+	0    -1   -1   0
+$EndComp
+Wire Wire Line
+	3950 5250 3800 5250
+Wire Wire Line
+	3500 5250 3000 5250
+Wire Wire Line
+	2850 5100 3050 5100
+Wire Wire Line
+	3050 4350 3050 5250
+Connection ~ 3050 5250
+Connection ~ 3050 5100
 $EndSCHEMATC
